File: hardware/braillebox/braillebox.kicad_sch (KiCad schematic)
At the start: 1 part, among them U1 XIAO-ESP32-S3-DIP

Commit message: Make circuit
Parts:
- added J1: PCA9685, Connector_PinSocket_2.54mm:PinSocket_1x06_P2.54mm_Vertical, symbol Connector:Conn_01x06_Socket
- added J2: Botão, TerminalBlock_Phoenix:TerminalBlock_Phoenix_MKDS-1,5-2_1x02_P5.00mm_Horizontal, symbol Connector:Conn_01x02_Socket
Connections:
- net +3.3V: now also J1.5 (Pin_5)
- net GND: now also J1.1 (Pin_1), J2.1 (Pin_1)
- net at U1.4 (GPIO4_A3_D3): now also J2.2 (Pin_2)
- net at U1.5 (GPIO5_A4_D4_SDA): now also J1.4 (Pin_4)
- net at U1.6 (GPIO6_A5_D5_SCL): now also J1.3 (Pin_3)
